File: choc/pcb/pcb.kicad_pcb (KiCad board)
At the start: 2 copper layers, 120 x 83 mm, 70 parts, among them SW1 Switch, SW10 Switch, SW11 Switch, SW12 Switch, SW13 Switch, SW14 Switch, SW15 Switch, SW16 Switch, SW17 Switch, SW18 Switch, SW19 Switch, SW2 Switch, SW3 Switch, SW4 Switch, SW5 Switch, SW6 Switch, SW7 Switch, SW8 Switch, SW9 Switch

Commit message: second
Parts:
- moved D19 21.9 mm to (128.5, 121.0), turned to 160 degrees
- moved D18 19.7 mm to (117.5, 119.0), turned to 170 degrees
- moved D17 18.0 mm to (99.5, 117.5)
- moved MCU1 1.00 mm to (50.0, 56.0)
- moved MCU2 1.00 mm to (50.0, 56.0)
- moved TRRS1 1.00 mm to (151.0, 44.5)
Changed lines of the file:
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@@
   )
   (footprint "zzkeeb:Connector_TRRS-reversible" (layer "F.Cu")
-    (at 151 43.5)
+    (at 151 44.5)
     (property "Sheetfile" "pcb.kicad_sch")
     (property "Sheetname" "")
@@
   )
   (footprint "zzkeeb:MCU_rp2040-zero-smd" (layer "F.Cu")
-    (at 49 56 90)
+    (at 50 56 90)
     (property "Sheetfile" "pcb.kicad_sch")
     (property "Sheetname" "")
@@
   )
   (footprint "zzkeeb:Diode_1N4148-SOD123-reversible-flip3d" (layer "B.Cu")
-    (at 125.5 101 180)
+    (at 117.5 119 170)
     (descr "Resitance 3 pas")
     (tags "R")
@@
     (property "row" "3")
     (attr through_hole)
-    (fp_text reference "D18" (at 0 1.5) (layer "B.SilkS") hide
+    (fp_text reference "D18" (at 0 1.5 -10) (layer "B.SilkS") hide
         (effects (font (size 0.9 0.9) (thickness 0.15) bold) (justify mirror))
     )
-    (fp_text value "D" (at -0.6 0) (layer "B.Fab") hide
+    (fp_text value "D" (at -0.6 0 -10) (layer "B.Fab") hide
         (effects (font (size 0.5 0.5) (thickness 0.125)) (justify mirror))
     )
-    (fp_text user "C${col}R${row}" (at 0 -1.5) (layer "B.SilkS")
+    (fp_text user "C${col}R${row}" (at 0 -1.5 -10) (layer "B.SilkS")
         (effects (font (size 0.9 0.9) (thickness 0.15)) (justify mirror))
     )
-    (fp_text user "C${col}R${row}" (at 0 -1.5) (layer "F.SilkS")
+    (fp_text user "C${col}R${row}" (at 0 -1.5 -10) (layer "F.SilkS")
         (effects (font (size 0.9 0.9) (thickness 0.15)))
     )
@@
     (fp_line (start 2.7 0.75) (end -2.95 0.75)
       (stroke (width 0.15) (type solid)) (layer "F.SilkS"))
-    (pad "1" smd rect (at -1.775 0 180) (size 1.3 0.95) (layers "F.Cu" "F.Paste" "F.Mask")
+    (pad "1" smd rect (at -1.775 0 170) (size 1.3 0.95) (layers "F.Cu" "F.Paste" "F.Mask")
       (net 20 "row3") (pinfunction "K") (pintype "passive"))
-    (pad "1" smd rect (at -1.775 0 180) (size 1.3 0.95) (layers "B.Cu" "B.Paste" "B.Mask")
+    (pad "1" smd rect (at -1.775 0 170) (size 1.3 0.95) (layers "B.Cu" "B.Paste" "B.Mask")
       (net 20 "row3") (pinfunction "K") (pintype "passive"))
-    (pad "2" smd rect (at 1.775 0 180) (size 1.3 0.95) (layers "F.Cu" "F.Paste" "F.Mask")
+    (pad "2" smd rect (at 1.775 0 170) (size 1.3 0.95) (layers "F.Cu" "F.Paste" "F.Mask")
       (net 32 "Net-(D18-A)") (pinfunction "A") (pintype "passive"))
-    (pad "2" smd rect (at 1.775 0 180) (size 1.3 0.95) (layers "B.Cu" "B.Paste" "B.Mask")
+    (pad "2" smd rect (at 1.775 0 170) (size 1.3 0.95) (layers "B.Cu" "B.Paste" "B.Mask")
       (net 32 "Net-(D18-A)") (pinfunction "A") (pintype "passive"))
     (model "${ZZKEEB}/lib/kbd/kicad-packages3D/kbd.3dshapes/D_SOD-123 Soldered.step"
@@
   )
   (footprint "zzkeeb:Diode_1N4148-SOD123-reversible-flip3d" (layer "B.Cu")
-    (at 144 105.5 180)
+    (at 128.5 121 160)
     (descr "Resitance 3 pas")
     (tags "R")
@@
     (property "row" "3")
     (attr through_hole)
-    (fp_text reference "D19" (at 0 1.5) (layer "B.SilkS") hide
+    (fp_text reference "D19" (at 0 1.5 -20) (layer "B.SilkS") hide
         (effects (font (size 0.9 0.9) (thickness 0.15) bold) (justify mirror))
     )
-    (fp_text value "D" (at -0.6 0) (layer "B.Fab") hide
+    (fp_text value "D" (at -0.6 0 -20) (layer "B.Fab") hide
         (effects (font (size 0.5 0.5) (thickness 0.125)) (justify mirror))
     )
-    (fp_text user "C${col}R${row}" (at 0 -1.5) (layer "B.SilkS")
+    (fp_text user "C${col}R${row}" (at 0 -1.5 -20) (layer "B.SilkS")
         (effects (font (size 0.9 0.9) (thickness 0.15)) (justify mirror))
     )
-    (fp_text user "C${col}R${row}" (at 0 -1.5) (layer "F.SilkS")
+    (fp_text user "C${col}R${row}" (at 0 -1.5 -20) (layer "F.SilkS")
         (effects (font (size 0.9 0.9) (thickness 0.15)))
     )
@@
     (fp_line (start 2.7 0.75) (end -2.95 0.75)
       (stroke (width 0.15) (type solid)) (layer "F.SilkS"))
-    (pad "1" smd rect (at -1.775 0 180) (size 1.3 0.95) (layers "F.Cu" "F.Paste" "F.Mask")
+    (pad "1" smd rect (at -1.775 0 160) (size 1.3 0.95) (layers "F.Cu" "F.Paste" "F.Mask")
       (net 20 "row3") (pinfunction "K") (pintype "passive"))
-    (pad "1" smd rect (at -1.775 0 180) (size 1.3 0.95) (layers "B.Cu" "B.Paste" "B.Mask")
+    (pad "1" smd rect (at -1.775 0 160) (size 1.3 0.95) (layers "B.Cu" "B.Paste" "B.Mask")
       (net 20 "row3") (pinfunction "K") (pintype "passive"))
-    (pad "2" smd rect (at 1.775 0 180) (size 1.3 0.95) (layers "F.Cu" "F.Paste" "F.Mask")
+    (pad "2" smd rect (at 1.775 0 160) (size 1.3 0.95) (layers "F.Cu" "F.Paste" "F.Mask")
       (net 33 "Net-(D19-A)") (pinfunction "A") (pintype "passive"))
-    (pad "2" smd rect (at 1.775 0 180) (size 1.3 0.95) (layers "B.Cu" "B.Paste" "B.Mask")
+    (pad "2" smd rect (at 1.775 0 160) (size 1.3 0.95) (layers "B.Cu" "B.Paste" "B.Mask")
       (net 33 "Net-(D19-A)") (pinfunction "A") (pintype "passive"))
     (model "${ZZKEEB}/lib/kbd/kicad-packages3D/kbd.3dshapes/D_SOD-123 Soldered.step"
@@
   )
   (footprint "zzkeeb:MCU_rp2040-zero-smd" (layer "B.Cu")
-    (at 49 56 -90)
+    (at 50 56 -90)
     (property "Sheetfile" "pcb.kicad_sch")
     (property "Sheetname" "")
@@
   )
   (footprint "zzkeeb:Diode_1N4148-SOD123-reversible-flip3d" (layer "B.Cu")
-    (at 99.5 99.5 180)
+    (at 99.5 117.5 180)
     (descr "Resitance 3 pas")
     (tags "R")

Commit message: third
Parts:
- moved H2 29.0 mm to (70.5, 122.0)
- moved H3 18.5 mm to (40.5, 103.5)
- moved FiveWay1 3.04 mm to (77.0, 114.5)
Other:
- outline, holes or cut-outs redrawn
Changed lines of the file:
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@@
   )
   (footprint "zzkeeb:Hole_M2" (layer "F.Cu")
-    (at 40.5 122)
+    (at 40.5 103.5)
     (descr "Mounting Hole 2.2mm, no annular, M2")
     (tags "mounting hole 2.2mm no annular m2")
@@
   )
   (footprint "zzkeeb:Button_5way-reversible" (layer "F.Cu")
-    (at 76.5 111.5)
+    (at 77 114.5)
     (property "Sheetfile" "pcb.kicad_sch")
     (property "Sheetname" "")
@@
   )
   (footprint "zzkeeb:Hole_M2" (layer "F.Cu")
-    (at 99.5 122)
+    (at 70.5 122)
     (descr "Mounting Hole 2.2mm, no annular, M2")
     (tags "mounting hole 2.2mm no annular m2")
@@
   (gr_line (start 157 44.5) (end 157 123.5)
     (stroke (width 0.1) (type default)) (layer "Edge.Cuts"))
+  (gr_arc (start 69 125.5) (mid 67.585786 124.914214) (end 67 123.5)
+    (stroke (width 0.1) (type default)) (layer "Edge.Cuts"))
   (gr_line (start 37 50.5) (end 58 50.5)
     (stroke (width 0.1) (type default)) (layer "Edge.Cuts"))
-  (gr_line (start 37 123.5) (end 37 61.5)
+  (gr_line (start 37 105) (end 37 61.5)
     (stroke (width 0.1) (type default)) (layer "Edge.Cuts"))
   (gr_line (start 58 61.5) (end 37 61.5)
@@
   (gr_line (start 58 50.5) (end 58 61.5)
     (stroke (width 0.1) (type default)) (layer "Edge.Cuts"))
+  (gr_line (start 67 107) (end 67 123.5)
+    (stroke (width 0.1) (type default)) (layer "Edge.Cuts"))
   (gr_arc (start 37 44.5) (mid 37.585786 43.085786) (end 39 42.5)
     (stroke (width 0.1) (type default)) (layer "Edge.Cuts"))
-  (gr_line (start 155 125.5) (end 39 125.5)
+  (gr_line (start 39 107) (end 67 107)
+    (stroke (width 0.1) (type default)) (layer "Edge.Cuts"))
+  (gr_line (start 155 125.5) (end 69 125.5)
     (stroke (width 0.1) (type default)) (layer "Edge.Cuts"))
   (gr_line (start 37 50.5) (end 37 44.5)
     (stroke (width 0.1) (type default)) (layer "Edge.Cuts"))
-  (gr_arc (start 39 125.5) (mid 37.585786 124.914214) (end 37 123.5)
+  (gr_arc (start 39 107) (mid 37.585786 106.414214) (end 37 105)
     (stroke (width 0.1) (type default)) (layer "Edge.Cuts"))
 )

Commit message: forth
Parts:
- removed the D5 at (47.5, 84.5)
- removed H6: MountingHole, zzkeeb:Hole_M2
- removed TRRS1: AudioJack4, zzkeeb:Connector_TRRS-reversible
- moved H5 38.0 mm to (153.0, 45.5)
- moved D19 22.4 mm to (146.0, 107.0)
- moved USB1 17.0 mm to (157.0, 54.5)
- moved USB2 17.0 mm to (157.0, 54.5)
- moved H4 6.08 mm to (71.0, 45.5)
- moved FiveWay1 2.12 mm to (78.5, 113.0)
- moved MCU1 1.50 mm to (50.0, 54.5)
- moved MCU2 1.50 mm to (50.0, 54.5)
- moved H1 0.71 mm to (153.0, 121.5)
- moved H2 0.71 mm to (71.0, 121.5)
- moved H3 0.50 mm to (41.0, 103.5)
Other:
- board size 120 x 83 mm -> 120 x 84 mm

Commit message: small updates
Parts:
- moved H3 1.00 mm to (40.0, 103.5)
- moved MCU1 1.00 mm to (49.0, 54.5)
- moved MCU2 1.00 mm to (49.0, 54.5)
Other:
- board size 120 x 84 mm -> 121 x 84 mm
Changed lines of the file:
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@@
   )
   (footprint "zzkeeb:Hole_M2" (layer "F.Cu")
-    (at 41 103.5)
+    (at 40 103.5)
     (descr "Mounting Hole 2.2mm, no annular, M2")
     (tags "mounting hole 2.2mm no annular m2")
@@
       (net 26 "col0") (pinfunction "6") (pintype "passive"))
     (model "${ZZKEEB}/models/5-WayTactileButton10mmTHT.stp"
-      (offset (xyz 5 5 0))
+      (offset (xyz 5.1 5.1 0.1))
       (scale (xyz 1 1 1))
       (rotate (xyz 0 0 -180))
     )
-    (model "${ZZKEEB}/models/5-way-concave-short.step"
+    (model "${ZZKEEB}/models/5-way-concave-short.step" hide
       (offset (xyz 0 0 6.5))
       (scale (xyz 1 1 1))
@@
   )
   (footprint "zzkeeb:MCU_rp2040-zero-smd" (layer "F.Cu")
-    (at 50 54.5 90)
+    (at 49 54.5 90)
     (property "Sheetfile" "pcb.kicad_sch")
     (property "Sheetname" "")
@@
   )
   (footprint "zzkeeb:MCU_rp2040-zero-smd" (layer "B.Cu")
-    (at 50 54.5 -90)
+    (at 49 54.5 -90)
     (property "Sheetfile" "pcb.kicad_sch")
     (property "Sheetname" "")
@@
   (gr_arc (start 69 125.5) (mid 67.585786 124.914214) (end 67 123.5)
     (stroke (width 0.1) (type default)) (layer "Edge.Cuts"))
-  (gr_line (start 37 49) (end 59 49)
+  (gr_line (start 36 49) (end 58 49)
     (stroke (width 0.1) (type default)) (layer "Edge.Cuts"))
-  (gr_line (start 37 105.5) (end 37 60)
+  (gr_line (start 36 105.5) (end 36 60)
     (stroke (width 0.1) (type default)) (layer "Edge.Cuts"))
-  (gr_line (start 59 60) (end 37 60)
+  (gr_line (start 58 60) (end 36 60)
     (stroke (width 0.1) (type default)) (layer "Edge.Cuts"))
-  (gr_line (start 39 41.5) (end 155 41.5)
+  (gr_line (start 38 41.5) (end 155 41.5)
     (stroke (width 0.1) (type default)) (layer "Edge.Cuts"))
   (gr_arc (start 157 123.5) (mid 156.414214 124.914214) (end 155 125.5)
     (stroke (width 0.1) (type default)) (layer "Edge.Cuts"))
-  (gr_line (start 59 49) (end 59 60)
+  (gr_line (start 58 49) (end 58 60)
     (stroke (width 0.1) (type default)) (layer "Edge.Cuts"))
   (gr_line (start 67 107.5) (end 67 123.5)
     (stroke (width 0.1) (type default)) (layer "Edge.Cuts"))
-  (gr_arc (start 37 43.5) (mid 37.585786 42.085786) (end 39 41.5)
+  (gr_arc (start 36 43.5) (mid 36.585786 42.085786) (end 38 41.5)
     (stroke (width 0.1) (type default)) (layer "Edge.Cuts"))
-  (gr_line (start 39 107.5) (end 67 107.5)
+  (gr_line (start 38 107.5) (end 67 107.5)
     (stroke (width 0.1) (type default)) (layer "Edge.Cuts"))
   (gr_line (start 155 125.5) (end 69 125.5)
     (stroke (width 0.1) (type default)) (layer "Edge.Cuts"))
-  (gr_line (start 37 49) (end 37 43.5)
+  (gr_line (start 36 49) (end 36 43.5)
     (stroke (width 0.1) (type default)) (layer "Edge.Cuts"))
-  (gr_arc (start 39 107.5) (mid 37.585786 106.914214) (end 37 105.5)
+  (gr_arc (start 38 107.5) (mid 36.585786 106.914214) (end 36 105.5)
     (stroke (width 0.1) (type default)) (layer "Edge.Cuts"))
 )

Commit message: fifth
Parts:
- USB1: moved to F.Cu
- USB2: moved to B.Cu
- moved H3 8.94 mm to (48.0, 107.5)
- moved H1 8.00 mm to (153.0, 113.5)
- moved H5 8.00 mm to (145.0, 45.5)
- moved H2 5.00 mm to (76.0, 121.5)
- moved H4 3.00 mm to (68.0, 45.5)
- turned USB1 to 90 degrees
- turned USB2 to -90 degrees
Other:
- outline, holes or cut-outs redrawn

Commit message: sixth
Parts:
- moved H2 32.9 mm to (100.5, 99.5)
- moved D18 29.2 mm to (142.5, 104.0)
- moved D17 22.6 mm to (115.5, 101.5)
- moved FiveWay1 18.8 mm to (97.0, 109.5)
- moved LED17 18.6 mm to (158.0, 112.1)
- moved LED18 18.6 mm to (138.4, 106.9)
- moved LED19 18.6 mm to (118.0, 105.3)
- moved SW17 18.6 mm to (118.0, 110.0)
- moved SW18 18.6 mm to (137.5, 111.5)
- moved SW19 18.6 mm to (156.5, 116.5)
- moved H1 14.0 mm to (153.0, 99.5)
- moved D19 4.74 mm to (150.5, 105.5)
- moved D15 4.00 mm to (123.5, 99.5)
- moved D16 4.00 mm to (133.5, 101.5)
- moved H3 0.17 mm to (48.0, 107.7)
Other:
- board size 121 x 84 mm -> 134.8 x 88.7 mm

Commit message: v1.0
Connections:
- LED19 pad 2: LED_OUT -> unconnected-(LED19-DOUT-Pad2)
Routing:
- net VCC: track 0.00 -> 529.2 mm, vias 0 -> 22
- net col4: track 0.00 -> 291.6 mm, vias 0 -> 6
- net TX: track 0.00 -> 285.0 mm, vias 0 -> 3
- net RX: track 0.00 -> 284.8 mm, vias 0 -> 3
- net col5: track 0.00 -> 276.5 mm, vias 0 -> 6
- net col3: track 0.00 -> 242.0 mm, vias 0 -> 6
- net row3: track 0.00 -> 161.3 mm, vias 0 -> 5
- net row2: track 0.00 -> 157.6 mm, vias 0 -> 8
- net row1: track 0.00 -> 155.1 mm, vias 0 -> 8
- net col0: track 0.00 -> 152.4 mm, vias 0 -> 3
- net col2: track 0.00 -> 151.1 mm, vias 0 -> 4
- net col1: track 0.00 -> 122.3 mm, vias 0 -> 4
- net row0: track 0.00 -> 109.8 mm, vias 0 -> 6
- net row4: track 0.00 -> 101.7 mm, vias 0 -> 1
- net LED: track 0.00 -> 74.3 mm, vias 0 -> 2
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- added copper zone on B.Cu, net GND
- added copper zone on F.Cu, net GND
Other:
- board text added: "bigga"
- board text added: "github.com/zzeneg/bigga"
- board text added: "v1.0"
