File: choc/pcb/pcb.kicad_sch (KiCad schematic)
At the start: 69 parts, among them SW10 Switch, SW11 Switch, SW12 Switch, SW13 Switch, SW14 Switch, SW15 Switch, SW18 Switch, SW19 Switch, SW3 Switch, SW4 Switch, SW5 Switch, SW6 Switch, SW7 Switch, SW8 Switch, SW9 Switch

Commit message: forth
Parts:
- removed H6: MountingHole, zzkeeb:Hole_M2, symbol Mechanical:MountingHole
- removed TRRS1: AudioJack4, zzkeeb:Connector_TRRS-reversible, symbol Connector_Audio:AudioJack4
Changed lines of the file:
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@@
-    (stroke (width 0) (type default))
-  )
-  (wire (pts (xy 148.59 41.91) (xy 151.13 41.91))
     (stroke (width 0) (type default))
   )
@@
     (stroke (width 0) (type default))
   )
-  (wire (pts (xy 148.59 39.37) (xy 148.59 41.91))
-    (stroke (width 0) (type default))
-  )
   (wire (pts (xy 133.35 69.85) (xy 133.35 78.74))
     (stroke (width 0) (type default))
@@
   )
   (wire (pts (xy 26.67 87.63) (xy 64.77 87.63))
-    (stroke (width 0) (type default))
-  )
-  (wire (pts (xy 148.59 36.83) (xy 156.21 36.83))
     (stroke (width 0) (type default))
   )
@@
     )
   )
-  (global_label "RX" (shape input) (at 148.59 34.29 0) (fields_autoplaced)
-    (effects (font (size 1.27 1.27)) (justify left))
-    (property "Intersheetrefs" "${INTERSHEET_REFS}" (at 153.4826 34.2106 0)
-      (effects (font (size 1.27 1.27)) (justify left) hide)
-    )
-  )
   (global_label "col2" (shape input) (at 116.84 44.45 0) (fields_autoplaced)
     (effects (font (size 1.27 1.27)) (justify left))
@@
     )
   )
-  (global_label "TX" (shape input) (at 148.59 31.75 0) (fields_autoplaced)
-    (effects (font (size 1.27 1.27)) (justify left))
-    (property "Intersheetrefs" "${INTERSHEET_REFS}" (at 153.1802 31.6706 0)
-      (effects (font (size 1.27 1.27)) (justify left) hide)
-    )
-  )
   (global_label "col4" (shape input) (at 58.42 41.91 0) (fields_autoplaced)
     (effects (font (size 1.27 1.27)) (justify left))
@@
         (path "/ebd24df5-909b-47ae-ba78-ebcdd375bb76"
           (reference "LED18") (unit 1)
-        )
-      )
-    )
-  )
-  (symbol (lib_id "power:GND") (at 156.21 36.83 0) (mirror y) (unit 1)
-    (in_bom yes) (on_board yes) (dnp no)
-    (property "Reference" "#PWR03" (at 156.21 43.18 0)
-      (effects (font (size 1.27 1.27)) hide)
-    )
-    (property "Value" "GND" (at 156.21 40.64 0)
-      (effects (font (size 1.27 1.27)))
-    )
-    (property "Footprint" "" (at 156.21 36.83 0)
-      (effects (font (size 1.27 1.27)) hide)
-    )
-    (property "Datasheet" "" (at 156.21 36.83 0)
-      (effects (font (size 1.27 1.27)) hide)
-    )
-    (pin "1")
-    (instances
-      (project "pcb"
-        (path "/5689f24b-6eca-4ca4-9c6c-dd56b6ced5a9"
-          (reference "#PWR03") (unit 1)
-        )
-      )
-      (project "pcb"
-        (path "/ebd24df5-909b-47ae-ba78-ebcdd375bb76"
-          (reference "#PWR012") (unit 1)
         )
       )
@@
         (path "/ebd24df5-909b-47ae-ba78-ebcdd375bb76"
           (reference "#PWR020") (unit 1)
-        )
-      )
-    )
-  )
-  (symbol (lib_id "Connector_Audio:AudioJack4") (at 143.51 34.29 0) (unit 1)
-    (in_bom yes) (on_board yes) (dnp no)
-    (property "Reference" "TRRS1" (at 143.51 25.4 0)
-      (effects (font (size 1.27 1.27)))
-    )
-    (property "Value" "AudioJack4" (at 143.51 27.94 0)
-      (effects (font (size 1.27 1.27)))
-    )
-    (property "Footprint" "zzkeeb:Connector_TRRS-reversible" (at 143.51 34.29 0)
-      (effects (font (size 1.27 1.27)) hide)
-    )
-    (property "Datasheet" "~" (at 143.51 34.29 0)
-      (effects (font (size 1.27 1.27)) hide)
-    )
-    (pin "R1")
-    (pin "R2")
-    (pin "S")
-    (pin "T")
-    (instances
-      (project "pcb"
-        (path "/5689f24b-6eca-4ca4-9c6c-dd56b6ced5a9"
-          (reference "TRRS1") (unit 1)
-        )
-      )
-      (project "pcb"
-        (path "/ebd24df5-909b-47ae-ba78-ebcdd375bb76"
-          (reference "TRRS1") (unit 1)
         )
       )
@@
     )
   )
-  (symbol (lib_id "Mechanical:MountingHole") (at 31.75 191.77 0) (unit 1)
-    (in_bom yes) (on_board yes) (dnp no) (fields_autoplaced)
-    (property "Reference" "H6" (at 34.29 190.4999 0)
-      (effects (font (size 1.27 1.27)) (justify left))
-    )
-    (property "Value" "MountingHole" (at 34.29 193.0399 0)
-      (effects (font (size 1.27 1.27)) (justify left))
-    )
-    (property "Footprint" "zzkeeb:Hole_M2" (at 31.75 191.77 0)
-      (effects (font (size 1.27 1.27)) hide)
-    )
-    (property "Datasheet" "~" (at 31.75 191.77 0)
-      (effects (font (size 1.27 1.27)) hide)
-    )
-    (instances
-      (project "pcb"
-        (path "/ebd24df5-909b-47ae-ba78-ebcdd375bb76"
-          (reference "H6") (unit 1)
-        )
-      )
-    )
-  )
   (symbol (lib_id "zzkeeb:LED_SK6812MINI-E") (at 204.47 128.27 0) (unit 1)
     (in_bom yes) (on_board yes) (dnp no)
@@
         )
       )
-    )
-  )
-  (symbol (lib_id "power:VCC") (at 151.13 41.91 0) (unit 1)
-    (in_bom yes) (on_board yes) (dnp no)
-    (property "Reference" "#PWR02" (at 151.13 45.72 0)
-      (effects (font (size 1.27 1.27)) hide)
-    )
-    (property "Value" "VCC" (at 151.13 38.1 0)
-      (effects (font (size 1.27 1.27)))
-    )
-    (property "Footprint" "" (at 151.13 41.91 0)
-      (effects (font (size 1.27 1.27)) hide)
-    )
-    (property "Datasheet" "" (at 151.13 41.91 0)
-      (effects (font (size 1.27 1.27)) hide)
-    )
-    (pin "1")
-    (instances
-      (project "pcb"
-        (path "/5689f24b-6eca-4ca4-9c6c-dd56b6ced5a9"
-          (reference "#PWR02") (unit 1)
-        )
-      )
-      (project "pcb"
-        (path "/ebd24df5-909b-47ae-ba78-ebcdd375bb76"
-          (reference "#PWR013") (unit 1)
-        )
-      )

Commit message: v1.0
Connections:
- net LED_OUT: no longer names the net of LED19.2 (DOUT)
- no-connect marks 24 -> 25
Changed lines of the file:
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@@
   (no_connect (at 58.42 31.75))
   (no_connect (at 237.49 35.56))
+  (no_connect (at 227.33 151.13))
   (no_connect (at 191.77 49.53))
   (no_connect (at 33.02 34.29))
@@
       (effects (font (size 1.27 1.27)) (justify left) hide)
     )
-  )
-  (global_label "LED_OUT" (shape input) (at 227.33 151.13 0) (fields_autoplaced)
-    (effects (font (size 1.27 1.27)) (justify left))
-    (property "Intersheetrefs" "${INTERSHEET_REFS}" (at 238.2791 151.13 0)
-      (effects (font (size 1.27 1.27)) (justify left) hide)
-    )
